File: pcb/usb-hub-2-electric-boogaloo.kicad_pcb (KiCad board)
At the start: 2 copper layers, 55 x 24.9 mm, 47 parts, among them U1 GL823K-HCY04, U2 SL2.1S

Commit message: update rev and add 3D back image
Other:
- board text added: "Another USB Hub SL2.1S Micro SD 2x USB-C 1x USB-A USB-C Upstream"
- board text added: "REV.3"
- board text removed: "Another USB Hub SL2.1S Micro SD 2x USB-C 1x USB-A USB-C Receptacle (no need for another cable *cough cough*)"
- board text removed: "REV.1"
Changed lines of the file:
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@@
 		)
 	)
-	(gr_text "REV.1"
+	(gr_text "REV.3"
 		(at 135.21 80.43 0)
 		(layer "F.SilkS")
@@
 		)
 	)
-	(gr_text "Another USB Hub\nSL2.1S\nMicro SD\n2x USB-C\n1x USB-A\nUSB-C Receptacle \n(no need for another cable *cough cough*)"
-		(at 127 75.3 0)
+	(gr_text "Another USB Hub\nSL2.1S\nMicro SD\n2x USB-C\n1x USB-A\nUSB-C Upstream"
+		(at 127.508 73.66 0)
 		(layer "B.SilkS")
 		(effects
